File: PCB/KiCAD/lcr/codec.kicad_sch (KiCad schematic)
At the start: 5 parts, among them U3 CS4272

Commit message: PCB Files
Parts:
- added C11, C13: 120p, Capacitor_SMD:C_0805_2012Metric, symbol Device:C
- added C12, C47, C49: 1u, Capacitor_SMD:C_0805_2012Metric, symbol Device:C
- added C14, C15: 33p, Capacitor_SMD:C_0805_2012Metric, symbol Device:C
- added C44: 47u, Capacitor_SMD:CP_Elec_5x5.9, symbol Device:C_US
- added C46, C48: .1u, Capacitor_SMD:C_0805_2012Metric, symbol Device:C
- added R19, R20: 5.1k, Resistor_SMD:R_0805_2012Metric, symbol Device:R_US
- added R21, R24: 8.2k, Resistor_SMD:R_0805_2012Metric, symbol Device:R_US
- added R22, R23: 10k, Resistor_SMD:R_0805_2012Metric, symbol Device:R_US
- added TP5, TP6, TP7: TestPoint, Others:testpoint_0805, symbol Connector:TestPoint
- added U17: TLV9162IDR, Package_SO:SOIC-8_3.9x4.9mm_P1.27mm, symbol Amplifiers:TLV9162IDR
- added Y1: Crystal, Crystal:Crystal_SMD_ECS_CSM3X-2Pin_7.6x4.1mm, symbol Device:Crystal
- C6: value 47u -> 1u; footprint (none) -> Capacitor_SMD:C_0805_2012Metric; KiLib_Generator (none) -> SMD_2terminal_chip_molded
- C7, C8, C9: footprint (none) -> Capacitor_SMD:C_0805_2012Metric; KiLib_Generator (none) -> SMD_2terminal_chip_molded
- U3: KiLib_Generator (none) -> package/gullwing
Connections:
- net +3.3V: now also C46.2, C47.2
- net +5VA: now also C48.2, C49.2
- net GND: now also U3.13 (AD0/~{CS}(I2S/~{LJ})), C14.2, C15.2, C44.2, C46.1, C47.1, C48.1, C49.1
- net at C6.2, C7.2, U3.22 (FILT+): now also C44.1
- net at U3.1 (XT0): now also C14.1, Y1.2
- net SCL: now reaches U3.11 (SCL/CCLK(M0))
- net SDA: now reaches U3.12 (SDA/CDIN(M1))
- net CODEC_RST: now reaches U3.14 (~{RST})
- net VSNS_P: now reaches U3.16 (AINA-)
- net VSNS_N: now reaches U3.17 (AINA+)
- net ISNS_P: now reaches U3.18 (AINB+)
- net ISNS_N: now reaches U3.19 (AINB-)
- net at U3.2 (XTI): now also C15.1, Y1.1
- net at U3.24 (AOUTA-): now also R23.1, TP6.1
- net at U3.25 (AOUTA+): now also R22.1, TP5.1
- net MCLK: now reaches U3.3 (MCLK)
- net LRCLK: now reaches U3.4 (LRCK)
- net BCLK: now reaches U3.5 (SCLK)
- net SDIN: now reaches U3.6 (SDOUT(M/~{S}))
- net SDOUT: now reaches U3.7 (SDIN)
- new net: C12.1, R20.1, R21.1, R22.2
- new net: C11.2, R20.2, U17.6 (-)
- new net: C12.2, R19.1, R23.2, R24.2
- new net: C13.1, R19.2, U17.5 (+)
- new net SIG_OUT: C11.1, R21.2, TP7.1, U17.7
- new net VMID: C13.2, R24.1
Other:
- company: (none) -> Owen Ball
- moved on the sheet: C8, C9
