File: PCB/KiCAD/lcr/lcr.kicad_sch (KiCad schematic)
At the start: 28 parts, among them U1 OPA2365AIDR, U2 THS4561IDGKR

Commit message: PCB Files
Parts:
- removed D1: ESD9L5.0ST5G, symbol Device:D_Zener
- added C16, C17, C25, C26: C, Capacitor_SMD:C_0805_2012Metric, symbol Device:C
- added C27, C34, C35, C36, C37, C38, C39, C40, C41, C42, C43, C51: 100n, Capacitor_SMD:C_0805_2012Metric, symbol Device:C
- added C28, C29: 470p, Capacitor_SMD:C_0805_2012Metric, symbol Device:C
- added C30: 2.7n, Capacitor_SMD:C_0805_2012Metric, symbol Device:C
- added D10, D11, D8, D9: ESD7205, Package_TO_SOT_SMD:SOT-323_SC-70, symbol Power_Protection:SP0502BAJT
- added F1, F2, F3, F4: 1206L012WR, Fuse:Fuse_1206_3216Metric, symbol Device:Polyfuse
- added J1, J2, J3, J4: Conn_Coaxial, BNC_Amphenol_B6252HB-NPP3G-50_Horizontal, symbol Connector:Conn_Coaxial
- added JP1: Jumper_2_Open, Connector_PinHeader_2.54mm:PinHeader_1x02_P2.54mm_Vertical, symbol Jumper:Jumper_2_Open
- added R27, R32, R33, R39, R40, R42, R43: R_US, Resistor_SMD:R_0805_2012Metric, symbol Device:R_US
- added R28, R38: 100k, Resistor_SMD:R_0805_2012Metric, symbol Device:R_US
- added R29, R37, R58, R59: 10k, Resistor_SMD:R_0805_2012Metric, symbol Device:R_US
- added R30, R34, R36, R52, R53, R54, R55: 1k, Resistor_SMD:R_0805_2012Metric, symbol Device:R_US
- added R31, R35, R47, R51: 100, Resistor_SMD:R_0805_2012Metric, symbol Device:R_US
- added R41: 1M, Resistor_SMD:R_0805_2012Metric, symbol Device:R_US
- added R44, R48: 8.2k, Resistor_SMD:R_0805_2012Metric, symbol Device:R_US
- added R45, R49: 1.6k, Resistor_SMD:R_0805_2012Metric, symbol Device:R_US
- added R46, R50: 300, Resistor_SMD:R_0805_2012Metric, symbol Device:R_US
- added R56, R57: 22, Resistor_SMD:R_0805_2012Metric, symbol Device:R_US
- added TP1, TP10, TP11, TP2, TP3, TP4, TP8, TP9: TestPoint, Others:testpoint_0805, symbol Connector:TestPoint
- added U12, U9: DG2034EDQ, Others:MSOP-10_largecorner, symbol Muxes:DG2034EDQ-T1-GE3
- added U13: OPA2365AIDR, Package_SO:SOIC-8_3.9x4.9mm_P1.27mm, symbol Amplifiers:OPA2365AIDR
- added U14: DG4052EEQ, Package_SO:TSSOP-16_4.4x5mm_P0.65mm, symbol Muxes:DG4052EEQ-T1-GE3
- added U15: THS4561IDGKR, Package_SO:TSSOP-8_3x3mm_P0.65mm, symbol Amplifiers:THS4561IDGKR
- added U17: TLV9162IDR, Package_SO:SOIC-8_3.9x4.9mm_P1.27mm, symbol Amplifiers:TLV9162IDR
- added U7: TLV9161IDBVR, Package_TO_SOT_SMD:SOT-23-5, symbol Amplifiers:TLV9161IDBVR
- C1, C10, C2, C5: footprint (none) -> Capacitor_SMD:C_0805_2012Metric; KiLib_Generator (none) -> SMD_2terminal_chip_molded
- C3, C4: value C -> 470p; footprint (none) -> Capacitor_SMD:C_0805_2012Metric; KiLib_Generator (none) -> SMD_2terminal_chip_molded
- R1, R8: value R_US -> 8.2k; footprint (none) -> Resistor_SMD:R_0805_2012Metric; KiLib_Generator (none) -> SMD_2terminal_chip_molded
- R10, R11, R12, R9: footprint (none) -> Resistor_SMD:R_0805_2012Metric; KiLib_Generator (none) -> SMD_2terminal_chip_molded
- R13, R14, R15: value R_US -> 1k; footprint (none) -> Resistor_SMD:R_0805_2012Metric; KiLib_Generator (none) -> SMD_2terminal_chip_molded
- R16, R18: value R_US -> 22; footprint (none) -> Resistor_SMD:R_0805_2012Metric; KiLib_Generator (none) -> SMD_2terminal_chip_molded
- R17: value R_US -> 1M; footprint (none) -> Resistor_SMD:R_0805_2012Metric; KiLib_Generator (none) -> SMD_2terminal_chip_molded
- R2, R7: value R_US -> 1.6k; footprint (none) -> Resistor_SMD:R_0805_2012Metric; KiLib_Generator (none) -> SMD_2terminal_chip_molded
- R3, R6: value R_US -> 300; footprint (none) -> Resistor_SMD:R_0805_2012Metric; KiLib_Generator (none) -> SMD_2terminal_chip_molded
- R4, R5: value R_US -> 100; footprint (none) -> Resistor_SMD:R_0805_2012Metric; KiLib_Generator (none) -> SMD_2terminal_chip_molded
- U1: KiLib_Generator (none) -> package/gullwing
- U2: footprint Package_SO:VSSOP-8_3x3mm_P0.65mm -> Package_SO:TSSOP-8_3x3mm_P0.65mm
- U4: value (none) -> DG4052EEQ; footprint (none) -> Package_SO:TSSOP-16_4.4x5mm_P0.65mm; KiLib_Generator (none) -> package/gullwing
Connections:
- net +5VA: now also C34.2, C35.2, C36.2, C37.2, C38.2, C39.2, C40.2, C41.2, C42.2, C43.2, U12.5 (EN), U12.6 (V+), U13.8 (V+), U14.16 (V+), U15.3 (V_{S+}), U15.7 (~{PD}), U17.8 (V+), U7.5 (V+), U9.5 (EN), U9.6 (V+)
- net GND: now also U4.6 (EN), C27.1, C34.1, C35.1, C36.1, C37.1, C38.1, C39.1, C40.1, C41.1, C42.1, C43.1, C51.1, D10.2 (K), D10.3 (A), D11.2 (K), D11.3 (A), D8.2 (K), D8.3 (A), D9.2 (K), D9.3 (A), J1.2 (Ext), J2.2 (Ext), J3.2 (Ext), J4.2 (Ext), U12.3 (V-), U13.4 (V-), U14.6 (EN), U14.7 (V-), U14.8 (GND), U15.6 (V_{S-}), U17.4 (V-), U7.2 (V-), U9.3 (V-)
- net VCOM: now also C27.2, U15.2 (V_{OCM})
- net at C2.2, R1.1, R10.1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: now also R14.2, TP9.1; no longer R14.1
- net at C1.2, R11.1, R13.2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: now also TP8.1
- net ISNS_N: now reaches C5.1, R18.1
- net ISNS_N: now also R34.1, TP2.1; no longer R17.2
- net at C4.1, U2.1 (-): now also R14.1, R34.2; no longer R14.2, R17.1
- net at U1.3 (+): now also R32.1
- net at C3.1, R13.1, U2.8 (+): now also R15.2; no longer R15.1
- net ISNS_P: now reaches C5.2, R16.1
- net ISNS_P: now also R15.1, TP1.1; no longer R15.2
- net at U1.5 (+): now also R33.1
- net PGA_I_0: now reaches U4.10 (A)
- net PGA_I_1: now reaches U4.9 (B)
- new net: R38.1, U12.7 (S4)
- new net: R48.2, R49.1, U14.14 (X1)
- new net: R49.2, R50.1, U14.15 (X2)
- new net: C29.1, R53.1, R55.2, U15.1 (-)
- new net: C29.2, R57.2, U15.4
- new net: C17.2, R29.1, U9.4 (S3)
- new net: R35.1, U12.2 (S1)
- new net: R37.1, U12.4 (S3)
- new net: R36.1, U12.9 (S2)
- new net: C28.1, R52.1, R54.2, U15.8 (+)
- new net: C51.2, R27.1, U7.3 (+)
- new net: C26.2, R41.1, R43.2, R44.1, R53.2, TP10.1, U13.7, U14.1 (Y0)
- new net: R44.2, R45.1, U14.5 (Y1)
- new net: R50.2, R51.1, U14.11 (X3)
- new net: C25.2, R17.1, R42.1, R48.1, R52.2, TP11.1, U13.1, U14.12 (X0)
- new net: C25.1, R17.2, U13.2 (-), U14.13 (X)
- new net: R45.2, R46.1, U14.2 (Y2)
- new net: C26.1, R41.2, U13.6 (-), U14.3 (Y)
- new net: R46.2, R47.1, U14.4 (Y3)
- new net: R39.1, U13.3 (+)
- new net: R42.2, R43.1, R47.2, R51.2
- new net: D10.1 (K), F2.2, R39.2, R58.2
- new net: F1.1, J1.1 (In)
- new net: R40.1, U13.5 (+)
- new net: D9.1 (K), F3.2, R40.2, R59.1
- new net: F2.1, J2.1 (In)
- new net: F4.1, J4.1 (In)
- new net: R30.1, U9.9 (S2)
- new net: C28.2, R56.2, U15.5
- new net: F3.1, J3.1 (In)
- new net: R31.1, U9.2 (S1)
- new net: C16.2, R28.1, U9.7 (S4)
- new net PGA_V_0: U14.10 (A)
- new net PGA_V_1: U14.9 (B)
- new net RSEL_0: U12.1 (A0), U9.1 (A0)
- new net RSEL_1: U12.10 (A1), U9.10 (A1)
- new net SIG_OUT: U17.3 (+)
- new net TIA_FB: C16.1, C17.1, D8.1 (K), F4.2, R28.2, R29.2, R30.2, R31.2, R33.2, R59.2, U7.4 (-)
- new net TIA_OUT: R32.2, U7.1, U9.8 (COM)
- new net VMID: R27.2
- new net VSNS_N: C30.1, R55.1, R57.1, TP4.1
- new net VSNS_P: C30.2, R54.1, R56.1, TP3.1
- new net sig_buf: JP1.2 (B), U12.8 (COM), U17.1, U17.2 (-)
- new net sig_conn: D11.1 (K), F1.2, JP1.1 (A), R35.2, R36.2, R37.2, R38.2, R58.1
Other:
- company: (none) -> Owen Ball
- moved on the sheet: C1, C10, C2, C3, C5, R1, R10, R11, R12, R13, R16, R2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
