File: PCB/KiCAD/lcr/power.kicad_sch (KiCad schematic)
At the start: 24 parts, among them J6 Screw_Terminal_01x02, J7 Barrel_Jack_Switch, SW1 SW_SPST, U10 MC7805, U11 MC7805, U16 TLV9161IDBVR

Commit message: top level pcb routing
Parts:
- SW1: footprint (none) -> Connector_PinHeader_2.54mm:PinHeader_1x02_P2.54mm_Vertical
Connections:
- net GND: now also J6.1 (Pin_1); no longer J6.2 (Pin_2)
- net at J7.1, SW1.1 (A): now also J6.2 (Pin_2); no longer J6.1 (Pin_1)
Other:
- moved on the sheet: J6
Changed lines of the file:
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@@
+	(wire
+		(pts
+			(xy 40.64 106.68) (xy 50.8 106.68)
+		)
+		(stroke
+			(width 0)
+			(type default)
+		)
+	)
 	(wire
 		(pts
@@
 		(pts
 			(xy 156.21 127) (xy 156.21 129.54)
-		)
-		(stroke
-			(width 0)
-			(type default)
-		)
-	)
-	(wire
-		(pts
-			(xy 40.64 106.68) (xy 50.8 106.68)
 		)
 		(stroke
@@
 	(symbol
 		(lib_id "Connector:Screw_Terminal_01x02")
-		(at 35.56 106.68 180)
+		(at 35.56 104.14 0)
+		(mirror y)
 		(unit 1)
 		(body_style 1)
@@
 		(in_pos_files yes)
 		(dnp no)
-		(fields_autoplaced yes)
 		(property "Reference" "J6"
-			(at 35.56 97.79 0)
+			(at 35.56 113.03 0)
 			(show_name no)
 			(do_not_autoplace no)
@@
 		)
 		(property "Value" "Screw_Terminal_01x02"
-			(at 35.56 100.33 0)
+			(at 35.56 110.49 0)
 			(show_name no)
 			(do_not_autoplace no)
@@
 		)
 		(property "Footprint" "TerminalBlock_Phoenix_MKDS-1,5-2-5.08_1x02_P5.08mm_Horizontal"
-			(at 35.56 106.68 0)
+			(at 35.56 104.14 0)
 			(hide yes)
 			(show_name no)
@@
 		)
 		(property "Datasheet" ""
-			(at 35.56 106.68 0)
+			(at 35.56 104.14 0)
 			(hide yes)
 			(show_name no)
@@
 		)
 		(property "Description" "Generic screw terminal, single row, 01x02, script generated (kicad-library-utils/schlib/autogen/connector/)"
-			(at 35.56 106.68 0)
+			(at 35.56 104.14 0)
 			(hide yes)
 			(show_name no)
@@
 			)
 		)
-		(property "Footprint" ""
+		(property "Footprint" "Connector_PinHeader_2.54mm:PinHeader_1x02_P2.54mm_Vertical"
 			(at 62.23 87.63 0)
 			(hide yes)
