File: PCB/KiCAD/lcr_v2/codec.kicad_sch (KiCad schematic)
At the start: 27 parts, among them U17 TLV9162IDR, U3 CS4272, Y1 Crystal

Commit message: Rev 1 PCB files
Parts:
- C11, C13: value 120p -> 100p
- C12: value 1u -> 220p
- TP5: value TestPoint -> DAC+
- TP6: value TestPoint -> DAC-
- TP7: value TestPoint -> SIG
Changed lines of the file:
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@@
 			)
 		)
-		(property "Value" "TestPoint"
+		(property "Value" "SIG"
 			(at 255.27 84.3279 0)
 			(hide yes)
@@
 			)
 		)
-		(property "Value" "120p"
+		(property "Value" "100p"
 			(at 240.284 74.93 90)
 			(show_name no)
@@
 			)
 		)
-		(property "Value" "1u"
-			(at 215.646 89.408 0)
+		(property "Value" "220p"
+			(at 216.916 89.408 0)
 			(show_name no)
 			(do_not_autoplace no)
@@
 			)
 		)
-		(property "Value" "120p"
+		(property "Value" "100p"
 			(at 234.696 102.362 0)
 			(show_name no)
@@
 			)
 		)
-		(property "Value" "TestPoint"
-			(at 194.31 91.9479 0)
-			(hide yes)
+		(property "Value" "DAC-"
+			(at 189.992 86.868 0)
 			(show_name no)
 			(do_not_autoplace no)
@@
 			)
 		)
-		(property "Value" "TestPoint"
-			(at 194.31 81.7879 0)
-			(hide yes)
-			(show_name no)
-			(do_not_autoplace no)
+		(property "Value" "DAC+"
+			(at 189.738 76.454 0)
+			(show_name no)
+			(do_not_autoplace no)
