File: PCB/KiCAD/lcr_v2/lcr.kicad_pcb (KiCad board)
At the start: 4 copper layers, 100 x 100 mm, 167 parts, among them J1 Conn_Coaxial, J2 Conn_Coaxial, J3 Conn_Coaxial, J4 Conn_Coaxial, J5 Conn_01x08_Pin, J6 Screw_Terminal_01x02, J7 Barrel_Jack_Switch, J8 Conn_01x09_Pin, J9 Conn_01x14_Pin, SW1 SW_SPST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

Commit message: pcb layout
Parts:
- added D6: D_Schottky, Diode_SMD:D_0805_2012Metric, F.Cu at (174.5, 128.1)
- added J10: Conn_01x02_Pin, Connector_PinHeader_2.54mm:PinHeader_1x02_P2.54mm_Vertical, F.Cu at (176.9, 131.2)
- added Q1: DMG1012UWQ-7, Package_TO_SOT_SMD:SOT-323_SC-70, F.Cu at (163.9, 131.4)
- added Q2: DMG1012UWQ-7, Package_TO_SOT_SMD:SOT-323_SC-70, F.Cu at (170.6, 131.6)
- added R42: 1k, Resistor_SMD:R_0805_2012Metric, F.Cu at (177.1, 139.3)
- added R43: 10k, Resistor_SMD:R_0805_2012Metric, F.Cu at (163.9, 128.6)
- added R60: 1k, Resistor_SMD:R_0805_2012Metric, F.Cu at (163.9, 126.5)
- added R64: 1k, Resistor_SMD:R_0805_2012Metric, F.Cu at (170.6, 126.5)
- added R65: 10k, Resistor_SMD:R_0805_2012Metric, F.Cu at (170.6, 128.6)
- added R66: 0, Resistor_SMD:R_0805_2012Metric, F.Cu at (178.2, 128.1)
- added TP16: TestPoint, Others:testpoint_0805, F.Cu at (126.5, 130.0)
- J5: value Conn_01x08_Pin -> Conn_01x06_Pin; footprint Connector_PinHeader_2.54mm:PinHeader_1x08_P2.54mm_Vertical -> Connector_PinHeader_2.54mm:PinHeader_1x06_P2.54mm_Vertical
- moved BZ1 10.0 mm to (173.3, 140.2)
- moved J5 0.40 mm to (150.0, 79.2)
Connections:
- BZ1 pad 1: +5VD -> Net-(BZ1-+)
- BZ1 pad 2: unconnected-(BZ1---Pad2) -> Net-(BZ1--)
- J5 pad 2: /GPIO7 -> /GPIO5
- J5 pad 3: /GPIO6 -> /GPIO4
- J5 pad 4: /GPIO5 -> /GPIO3
- J5 pad 5: /GPIO4 -> /GPIO2
- J5 pad 6: /GPIO3 -> /GPIO1
- U5 pad 31: /GPIO7 -> /GPIO5
- U5 pad 32: /GPIO6 -> /GPIO4
- U5 pad 33: /GPIO5 -> /GPIO3
- U5 pad 36: /GPIO4 -> /BUZZ
- U5 pad 37: /GPIO3 -> /FAN_PWM
Routing:
- net /BUZZ: track 0.00 -> 54.7 mm, vias 0 -> 1
- net /FAN_PWM: track 0.00 -> 53.4 mm, vias 0 -> 1
- net +5VD: track 108.5 -> 119.5 mm, vias 2 -> 3
- net Net-(BZ1--): track 0.00 -> 8.65 mm
- net Net-(D6-A): track 0.00 -> 7.69 mm
- net Net-(D6-K): track 0.00 -> 5.12 mm
- net /GPIO2: track 6.89 -> 11.8 mm
- net /GPIO1: track 6.86 -> 11.8 mm
- net Net-(Q1-G): track 0.00 -> 4.88 mm
- net /GPIO7: track 4.42 -> 0.00 mm
- net /GPIO6: track 4.42 -> 0.00 mm
- net Net-(Q2-G): track 0.00 -> 4.32 mm
- net GND: track 87.3 -> 91.6 mm, vias 78 -> 81
- net Net-(BZ1-+): track 0.00 -> 3.81 mm
- net /GPIO4: track 6.87 -> 4.02 mm
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Other:
- board text added: "+"
- board text added: "16"
- board text added: "17"
- board text added: "39"
- board text added: "40"
- board text added: "41"
- board text added: "Owen Ball April 2026 Teensy LCR Rev 1"

Commit message: Rev 1 PCB files
Parts:
- removed D5: D_Schottky, Diode_SMD:Nexperia_CFP3_SOD-123W
- removed U9: DG2034EDQ, Others:MSOP-10_largecorner
- added C32: C, Capacitor_SMD:C_0805_2012Metric, F.Cu at (123.6, 132.7)
- added D1: 7.5V, Diode_SMD:Nexperia_CFP3_SOD-123W, F.Cu at (187.5, 119.2)
- added Q3: DMP3099L, Package_TO_SOT_SMD:SOT-23, F.Cu at (184.0, 119.5)
- added R67: 100k, Resistor_SMD:R_0805_2012Metric, F.Cu at (187.5, 123.4)
- added TP17: VMID, Others:testpoint_0805, F.Cu at (162.3, 94.7)
- C11, C13: value 120p -> 100p
- C12: value 1u -> 220p
- D3: footprint Diode_SMD:D_SOD-123F -> Diode_SMD:Nexperia_CFP3_SOD-123W
- R60, R64: value 1k -> 100
- TP1: value TestPoint -> ISNS+
- TP10: value TestPoint -> VPGA-
- TP11: value TestPoint -> VPGA+
- TP12: value TestPoint -> 5VA
- TP13: value TestPoint -> 5VD
- TP14: value TestPoint -> SCL
- TP15: value TestPoint -> SDA
- TP16: value TestPoint -> TIA
- TP2: value TestPoint -> ISNS-
- TP3: value TestPoint -> VSNS+
- TP4: value TestPoint -> VSNS-
- TP5: value TestPoint -> DAC+
- TP6: value TestPoint -> DAC-
- TP7: value TestPoint -> SIG
- TP8: value TestPoint -> IPGA+
- TP9: value TestPoint -> IPGA-
- moved SW1 1.30 mm to (184.6, 126.4)
Routing:
- net Net-(D1-A): track 0.00 -> 4.51 mm
- net +3.3V: track 99.3 -> 102.3 mm
- net VMID: track 80.1 -> 82.1 mm
- net Net-(Q3-D): track 3.03 -> 4.92 mm
- net GND: track 91.6 -> 92.9 mm, vias 81 -> 266
- net /DISP_CS: track 22.3 -> 21.5 mm
- net Net-(U3-AOUTA-): track 36.6 -> 37.2 mm
- net Net-(U3-AOUTA+): track 38.8 -> 39.3 mm
Other:
- board text added: "Owen Ball Rev 1, April 2026"
- board text added: "TeensyLCR"
- board text removed: "Owen Ball April 2026 Teensy LCR Rev 1"

Commit message: Initial firmware commit
Parts:
- added U9: DG2034EDQ, Others:MSOP-10_largecorner, F.Cu at (133.1, 139.5)
