File: PCB/KiCAD/lcr_v2/lcr.kicad_pcb (KiCad board)
At the start: 4 copper layers, 100 x 100 mm, 182 parts, among them J1 Conn_Coaxial, J10 Conn_01x02_Pin, J2 Conn_Coaxial, J3 Conn_Coaxial, J4 Conn_Coaxial, J5 Conn_01x06_Pin, J6 Screw_Terminal_01x02, J7 Barrel_Jack_Switch, J8 Conn_01x09_Pin, J9 Conn_01x14_Pin, Q1 DMG1012UWQ-7, Q2 DMG1012UWQ-7, Q3 DMP3099L, SW1 SW_SPST, U1 OPA2365AIDR, U10 MC7805, U11 MC7805, U12 DG2034EDQ, U13 OPA2365AIDR, U14 DG4052EEQ, U15 THS4561IDGKR, U16 TLV9161IDBVR, U17 TLV9162IDR, U2 THS4561IDGKR, U3 CS4272, U4 DG4052EEQ, U5 Teensy4.1_mainpins, U6 MCP9800Ax-xOT, U7 TLV9161IDBVR, U9 DG2034EDQ, Y1 Crystal

Commit message: Test code
Parts:
- C1, C16, C17, C2, C25, C26, C32: value C -> 1p
- C20, C21, C22, C24: value C -> 1u
- R32, R33, R39, R40: value R_US -> 0
Changed lines of the file:
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@@
 			)
 		)
-		(property "Value" "C"
+		(property "Value" "1u"
 			(at 0 1.68 0)
 			(layer "F.Fab")
@@
 			)
 		)
-		(property "Value" "R_US"
+		(property "Value" "0"
 			(at 0 1.65 0)
 			(layer "F.Fab")
@@
 			)
 		)
-		(property "Value" "R_US"
+		(property "Value" "0"
 			(at 0 1.65 0)
 			(layer "F.Fab")
@@
 			)
 		)
-		(property "Value" "C"
+		(property "Value" "1u"
 			(at 0 1.68 0)
 			(layer "F.Fab")
@@
 			)
 		)
-		(property "Value" "C"
+		(property "Value" "1p"
 			(at 0 1.68 0)
 			(layer "F.Fab")
@@
 			)
 		)
-		(property "Value" "C"
+		(property "Value" "1p"
 			(at 0 1.68 90)
 			(layer "F.Fab")
@@
 			)
 		)
-		(attr smd)
+		(attr smd dnp)
 		(duplicate_pad_numbers_are_jumpers no)
 		(fp_line
@@
 			)
 		)
-		(property "Value" "C"
+		(property "Value" "1p"
 			(at 0 1.68 0)
 			(layer "F.Fab")
@@
 			)
 		)
-		(property "Value" "C"
+		(property "Value" "1p"
 			(at 0 1.68 90)
 			(layer "F.Fab")
@@
 			)
 		)
-		(property "Value" "C"
+		(property "Value" "1p"
 			(at 0 1.68 0)
 			(layer "F.Fab")
@@
 			)
 		)
-		(property "Value" "R_US"
+		(property "Value" "0"
 			(at 0 1.65 0)
 			(layer "F.Fab")
@@
 			)
 		)
-		(property "Value" "R_US"
+		(property "Value" "0"
 			(at 0 1.65 0)
 			(layer "F.Fab")
@@
 			)
 		)
-		(property "Value" "C"
+		(property "Value" "1u"
 			(at 0 1.68 0)
 			(layer "F.Fab")
@@
 			)
 		)
-		(property "Value" "C"
+		(property "Value" "1u"
 			(at 0 1.68 0)
 			(layer "F.Fab")
@@
 			)
 		)
-		(property "Value" "C"
+		(property "Value" "1p"
 			(at 0 1.68 0)
 			(layer "F.Fab")
@@
 			)
 		)
-		(property "Value" "C"
+		(property "Value" "1p"
 			(at 0 1.68 0)
 			(layer "F.Fab")
