File: PCB/KiCAD/lcr_v2/teensy.kicad_sch (KiCad schematic)
At the start: 12 parts, among them J5 Conn_01x08_Pin, J8 Conn_01x09_Pin, J9 Conn_01x14_Pin, U5 Teensy4.1_mainpins, U6 MCP9800Ax-xOT

Commit message: pcb layout
Parts:
- removed J5: Conn_01x08_Pin, Connector_PinHeader_2.54mm:PinHeader_1x08_P2.54mm_Vertical, symbol Connector:Conn_01x08_Pin
- added D6: D_Schottky, Diode_SMD:D_0805_2012Metric, symbol Device:D_Schottky
- added J10: Conn_01x02_Pin, Connector_PinHeader_2.54mm:PinHeader_1x02_P2.54mm_Vertical, symbol Connector:Conn_01x02_Pin
- added J5: Conn_01x06_Pin, Connector_PinHeader_2.54mm:PinHeader_1x06_P2.54mm_Vertical, symbol Connector:Conn_01x06_Pin
- added Q1, Q2: DMG1012UWQ-7, Package_TO_SOT_SMD:SOT-323_SC-70, symbol FETs:DMG1012UWQ-7
- added R42, R60, R64: 1k, Resistor_SMD:R_0805_2012Metric, symbol Device:R_US
- added R43, R65: 10k, Resistor_SMD:R_0805_2012Metric, symbol Device:R_US
- added R66: 0, Resistor_SMD:R_0805_2012Metric, symbol Device:R_US
Connections:
- net GPIO6 is gone; now on net GPIO4: U5.32 (40_A16)
- net GPIO7 is gone; now on net GPIO5: U5.31 (39_MISO1_OUT1A)
- net +5VD: now also R42.1, R66.1; no longer BZ1.1 (+)
- net GND: now also J5.1 (Pin_1), Q1.2 (S), Q2.2 (S), R43.2, R65.2
- net GPIO1: now also J5.6 (Pin_6)
- net GPIO2: now also J5.5 (Pin_5)
- net GPIO3: now also U5.33 (41_A17), J5.4 (Pin_4); no longer U5.37 (15_A1_RX3_SPDIF_IN)
- net GPIO4: now also J5.3 (Pin_3); no longer U5.36 (14_A0_TX3_SPDIF_OUT)
- net GPIO5: now also J5.2 (Pin_2); no longer U5.33 (41_A17)
- net at BZ1.2 (-): now also Q1.3 (D)
- new net: Q1.1 (G), R43.1, R60.2
- new net: Q2.1 (G), R64.2, R65.1
- new net: D6.2 (A), J10.2 (Pin_2), Q2.3 (D)
- new net: BZ1.1 (+), R42.2
- new net: D6.1 (K), J10.1 (Pin_1), R66.2
- new net BUZZ: R60.1, U5.36 (14_A0_TX3_SPDIF_OUT)
- new net FAN_PWM: R64.1, U5.37 (15_A1_RX3_SPDIF_IN)
Other:
- note removed: "BUZZER?"
- note removed: "FAN HEADER"
- moved on the sheet: BZ1, C50, J8, J9, R25, R26, R63, TP14, TP15, U5, U6

Commit message: Rev 1 PCB files
Parts:
- R60, R64: value 1k -> 100
- TP14: value TestPoint -> SCL
- TP15: value TestPoint -> SDA
Other:
- note removed: "LED?"
Changed lines of the file:
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@@
 		(company "Owen Ball")
 	)
-	(text "LED?"
-		(exclude_from_sim no)
-		(at 65.786 78.232 0)
-		(effects
-			(font
-				(size 5.08 5.08)
-			)
-		)
-	)
 	(text "Display"
 		(exclude_from_sim no)
@@
 	)
 	(image
-		(at 165.1 203.2)
+		(at 118.11 190.5)
 		(data "iVBORw0KGgoAAAANSUhEUgAABX8AAALBCAYAAAAAtdJ9AAAABHNCSVQICAgIfAhkiAAAIABJREFU"
 			"eJzs3Xd4jecfx/H3OSeDWBlmFLF3qL1nae29qSJqd6KqVKnRVtufXVRtNWuvUnvvNkaIEVHUSCQh"
@@
 			)
 		)
-		(property "Value" "1k"
+		(property "Value" "100"
 			(at 196.85 140.97 0)
 			(show_name no)
@@
 			)
 		)
-		(property "Value" "TestPoint"
+		(property "Value" "SDA"
 			(at 223.52 61.4679 0)
 			(hide yes)
@@
 			)
 		)
-		(property "Value" "TestPoint"
+		(property "Value" "SCL"
 			(at 220.98 61.4679 0)
 			(hide yes)
@@
 			)
 		)
-		(property "Value" "1k"
+		(property "Value" "100"
 			(at 144.78 140.97 0)
 			(show_name no)
