File: PCB/KiCAD/lcr_v2/lcr.kicad_sch (KiCad schematic)
At the start: 103 parts, among them J1 Conn_Coaxial, J2 Conn_Coaxial, J3 Conn_Coaxial, J4 Conn_Coaxial, U1 OPA2365AIDR, U12 DG2034EDQ, U13 OPA2365AIDR, U14 DG4052EEQ, U15 THS4561IDGKR, U17 TLV9162IDR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

Commit message: pcb layout
Parts:
- added TP16: TestPoint, Others:testpoint_0805, symbol Connector:TestPoint
- J1, J2, J3, J4: footprint BNC_Amphenol_B6252HB-NPP3G-50_Horizontal -> Connector_Coaxial:BNC_Amphenol_B6252HB-NPP3G-50_Horizontal
Connections:
- net TIA_OUT: now also TP16.1
Other:
- note added: "HCUR"
- note added: "HPOT"
- note added: "LCUR"
- note added: "LPOT"
Changed lines of the file:
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@@
 		(company "Owen Ball")
 	)
+	(text "HCUR"
+		(exclude_from_sim no)
+		(at 96.774 79.248 0)
+		(effects
+			(font
+				(size 2.54 2.54)
+			)
+		)
+	)
+	(text "LPOT"
+		(exclude_from_sim no)
+		(at 96.1692 177.038 0)
+		(effects
+			(font
+				(size 2.54 2.54)
+			)
+		)
+	)
+	(text "HPOT"
+		(exclude_from_sim no)
+		(at 96.4716 131.318 0)
+		(effects
+			(font
+				(size 2.54 2.54)
+			)
+		)
+	)
+	(text "LCUR"
+		(exclude_from_sim no)
+		(at 96.4716 232.156 0)
+		(effects
+			(font
+				(size 2.54 2.54)
+			)
+		)
+	)
 	(junction
 		(at 421.64 284.48)
@@
 	)
 	(junction
+		(at 243.84 267.97)
+		(diameter 0)
+		(color 0 0 0 0)
+	)
+	(junction
 		(at 306.07 279.4)
 		(diameter 0)
@@
 	(wire
 		(pts
+			(xy 243.84 267.97) (xy 248.92 267.97)
+		)
+		(stroke
+			(width 0)
+			(type default)
+		)
+	)
+	(wire
+		(pts
 			(xy 384.81 288.29) (xy 384.81 271.78)
 		)
@@
 	(wire
 		(pts
-			(xy 238.76 267.97) (xy 248.92 267.97)
+			(xy 238.76 267.97) (xy 243.84 267.97)
 		)
 		(stroke
@@
 			)
 		)
-		(property "Footprint" "BNC_Amphenol_B6252HB-NPP3G-50_Horizontal"
+		(property "Footprint" "Connector_Coaxial:BNC_Amphenol_B6252HB-NPP3G-50_Horizontal"
 			(at 114.3 128.27 0)
 			(hide yes)
@@
 	)
 	(symbol
+		(lib_id "Connector:TestPoint")
+		(at 243.84 267.97 0)
+		(unit 1)
+		(body_style 1)
+		(exclude_from_sim no)
+		(in_bom yes)
+		(on_board yes)
+		(in_pos_files yes)
+		(dnp no)
+		(property "Reference" "TP16"
+			(at 242.316 262.636 0)
+			(show_name no)
+			(do_not_autoplace no)
+			(effects
+				(font
+					(size 1.27 1.27)
+				)
+				(justify left)
+			)
+		)
+		(property "Value" "TestPoint"
+			(at 246.38 265.9379 0)
+			(hide yes)
+			(show_name no)
+			(do_not_autoplace no)
+			(effects
+				(font
+					(size 1.27 1.27)
+				)
+				(justify left)
+			)
+		)
+		(property "Footprint" "Others:testpoint_0805"
+			(at 248.92 267.97 0)
+			(hide yes)
+			(show_name no)
+			(do_not_autoplace no)
+			(effects
+				(font
+					(size 1.27 1.27)
+				)
+			)
+		)
+		(property "Datasheet" ""
+			(at 248.92 267.97 0)
+			(hide yes)
+			(show_name no)
+			(do_not_autoplace no)
+			(effects
+				(font
+					(size 1.27 1.27)
+				)
+			)
+		)
+		(property "Description" "test point"
+			(at 243.84 267.97 0)
+			(hide yes)
+			(show_name no)
+			(do_not_autoplace no)
+			(effects
+				(font
+					(size 1.27 1.27)
+				)
+			)
+		)
+		(pin "1"
+		)
+		(instances
+			(project "lcr"
+				(path "/37326a55-d49a-46f0-b0ef-9b9ba0d9ea8b"
+					(reference "TP16")
+					(unit 1)
+				)
+			)
+		)
+	)
+	(symbol
 		(lib_id "Device:Polyfuse")
 		(at 129.54 128.27 90)
@@
 			)
 		)
-		(property "Footprint" "BNC_Amphenol_B6252HB-NPP3G-50_Horizontal"
+		(property "Footprint" "Connector_Coaxial:BNC_Amphenol_B6252HB-NPP3G-50_Horizontal"
 			(at 114.3 173.99 0)
 			(hide yes)
@@
 			)
 		)
-		(property "Footprint" "BNC_Amphenol_B6252HB-NPP3G-50_Horizontal"
+		(property "Footprint" "Connector_Coaxial:BNC_Amphenol_B6252HB-NPP3G-50_Horizontal"
 			(at 114.3 76.2 0)
 			(hide yes)
@@
 			)
 		)
-		(property "Footprint" "BNC_Amphenol_B6252HB-NPP3G-50_Horizontal"
+		(property "Footprint" "Connector_Coaxial:BNC_Amphenol_B6252HB-NPP3G-50_Horizontal"
 			(at 115.57 228.6 0)
 			(hide yes)

Commit message: Rev 1 PCB files
Parts:
- added C32: C, Capacitor_SMD:C_0805_2012Metric, symbol Device:C
- TP1: value TestPoint -> ISNS+
- TP10: value TestPoint -> VPGA-
- TP11: value TestPoint -> VPGA+
- TP16: value TestPoint -> TIA
- TP2: value TestPoint -> ISNS-
- TP3: value TestPoint -> VSNS+
- TP4: value TestPoint -> VSNS-
- TP8: value TestPoint -> IPGA+
- TP9: value TestPoint -> IPGA-
Connections:
- net TIA_FB: now also C32.1
- net TIA_OUT: now also C32.2
Other:
- moved on the sheet: C16, C17, C42, C43, R28, R29, R30, R31, U13C, U17C, U1C, U9

Commit message: Test code
Parts:
- C1, C16, C2, C25, C26, C32: value C -> 1p
- C17: value C -> 1p; now not fitted
- C51: value 100n -> 10u
- R27: value R_US -> 10k
- R32, R33, R39, R40: value R_US -> 0
Changed lines of the file:
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@@
 			)
 		)
-		(property "Value" "100n"
+		(property "Value" "10u"
 			(at 193.548 280.162 0)
 			(show_name no)
@@
 			)
 		)
-		(property "Value" "C"
+		(property "Value" "1p"
 			(at 297.434 146.05 90)
 			(show_name no)
@@
 			)
 		)
-		(property "Value" "C"
+		(property "Value" "1p"
 			(at 297.18 297.18 90)
 			(show_name no)
@@
 			)
 		)
-		(property "Value" "C"
+		(property "Value" "1p"
 			(at 297.18 157.48 90)
 			(show_name no)
@@
 		(on_board yes)
 		(in_pos_files yes)
-		(dnp no)
+		(dnp yes)
 		(property "Reference" "C17"
 			(at 195.072 233.68 90)
@@
 			)
 		)
-		(property "Value" "C"
+		(property "Value" "1p"
 			(at 200.66 233.68 90)
 			(show_name no)
@@
 		(dnp no)
 		(property "Reference" "R40"
-			(at 261.112 176.276 90)
+			(at 263.144 176.53 90)
 			(show_name no)
 			(do_not_autoplace no)
@@
 			)
 		)
-		(property "Value" "R_US"
-			(at 265.938 176.276 90)
+		(property "Value" "0"
+			(at 267.97 176.53 90)
 			(show_name no)
 			(do_not_autoplace no)
@@
 		(dnp no)
 		(property "Reference" "R39"
-			(at 261.112 130.556 90)
+			(at 262.89 130.81 90)
 			(show_name no)
 			(do_not_autoplace no)
@@
 			)
 		)
-		(property "Value" "R_US"
-			(at 265.938 130.556 90)
+		(property "Value" "0"
+			(at 267.97 130.81 90)
 			(show_name no)
 			(do_not_autoplace no)
@@
 			)
 		)
-		(property "Value" "R_US"
+		(property "Value" "10k"
 			(at 185.928 272.796 90)
 			(show_name no)
@@
 		(dnp no)
 		(property "Reference" "R33"
-			(at 261.112 315.976 90)
+			(at 263.398 316.23 90)
 			(show_name no)
 			(do_not_autoplace no)
@@
 			)
 		)
-		(property "Value" "R_US"
-			(at 265.938 315.976 90)
+		(property "Value" "0"
+			(at 268.224 316.23 90)
 			(show_name no)
 			(do_not_autoplace no)
@@
 			)
 		)
-		(property "Value" "C"
+		(property "Value" "1p"
 			(at 297.434 285.75 90)
 			(show_name no)
@@
 		(dnp no)
 		(property "Reference" "R32"
-			(at 261.112 270.256 90)
+			(at 263.398 270.51 90)
 			(show_name no)
 			(do_not_autoplace no)
@@
 			)
 		)
-		(property "Value" "R_US"
-			(at 265.938 270.256 90)
+		(property "Value" "0"
+			(at 268.224 270.51 90)
 			(show_name no)
 			(do_not_autoplace no)
@@
 			)
 		)
-		(property "Value" "C"
+		(property "Value" "1p"
 			(at 208.28 252.73 90)
 			(show_name no)
@@
 			)
 		)
-		(property "Value" "C"
+		(property "Value" "1p"
 			(at 200.66 243.84 90)
 			(show_name no)
