File: PCB/KiCAD/lcr_v2/power.kicad_sch (KiCad schematic)
At the start: 26 parts, among them J6 Screw_Terminal_01x02, J7 Barrel_Jack_Switch, SW1 SW_SPST, U10 MC7805, U11 MC7805, U16 TLV9161IDBVR

Commit message: pcb layout
Parts:
- J6: footprint TerminalBlock_Phoenix_MKDS-1,5-2-5.08_1x02_P5.08mm_Horizontal -> TerminalBlock_Phoenix:TerminalBlock_Phoenix_MKDS-1,5-2-5.08_1x02_P5.08mm_Horizontal
- J7: footprint BarrelJack_GCT_DCJ200-10-A_Horizontal -> Connector_BarrelJack:BarrelJack_GCT_DCJ200-10-A_Horizontal
Changed lines of the file:
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@@
 			)
 		)
-		(property "Footprint" "BarrelJack_GCT_DCJ200-10-A_Horizontal"
+		(property "Footprint" "Connector_BarrelJack:BarrelJack_GCT_DCJ200-10-A_Horizontal"
 			(at 35.56 91.186 0)
 			(hide yes)
@@
 			)
 		)
-		(property "Footprint" "TerminalBlock_Phoenix_MKDS-1,5-2-5.08_1x02_P5.08mm_Horizontal"
+		(property "Footprint" "TerminalBlock_Phoenix:TerminalBlock_Phoenix_MKDS-1,5-2-5.08_1x02_P5.08mm_Horizontal"
 			(at 35.56 106.68 0)
 			(hide yes)

Commit message: Rev 1 PCB files
Parts:
- removed D5: D_Schottky, Diode_SMD:Nexperia_CFP3_SOD-123W, symbol Device:D_Schottky
- added D1: 7.5V, Diode_SMD:Nexperia_CFP3_SOD-123W, symbol Device:D_Zener
- added Q3: DMP3099L, Package_TO_SOT_SMD:SOT-23, symbol Transistor_FET:DMP3099L
- added R67: 100k, Resistor_SMD:R_0805_2012Metric, symbol Device:R_US
- added TP17: VMID, Others:testpoint_0805, symbol Connector:TestPoint
- D3: footprint (none) -> Diode_SMD:Nexperia_CFP3_SOD-123W
- TP12: value TestPoint -> 5VA
- TP13: value TestPoint -> 5VD
Connections:
- net +12V: now also D1.1 (K), Q3.2 (S)
- net GND: now also R67.2
- net VMID: now also TP17.1
- net at SW1.2 (B): now also Q3.3 (D)
- new net: D1.2 (A), Q3.1 (G), R67.1
Other:
- moved on the sheet: C18, C19, C20, C21, C22, C23, C24, C33, C45, D3, D4, H1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

Commit message: Test code
Parts:
- C20, C21, C22, C24: value C -> 1u
- R67: value 100k -> 10k
Changed lines of the file:
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@@
 			)
 		)
-		(property "Value" "100k"
+		(property "Value" "10k"
 			(at 87.63 101.6 0)
 			(show_name no)
@@
 			)
 		)
-		(property "Value" "C"
+		(property "Value" "1u"
 			(at 162.56 125.7299 0)
 			(show_name no)
@@
 			)
 		)
-		(property "Value" "C"
+		(property "Value" "1u"
 			(at 132.08 82.5499 0)
 			(show_name no)
@@
 			)
 		)
-		(property "Value" "C"
+		(property "Value" "1u"
 			(at 162.56 82.5499 0)
 			(show_name no)
@@
 			)
 		)
-		(property "Value" "C"
+		(property "Value" "1u"
 			(at 132.08 125.7299 0)
 			(show_name no)
